File: Hardware/BT-5/BT-5.brd (EAGLE design)
At the start: 95 x 20 mm, 82 parts, among them J1 CORTEX_DEBUG_PTH, J2 AVR_SPI_PROG_3X22X3_LOCK, J5 JST_ZH_2PIN, U1 ATMEGA1284P-AU, U2 TPS61200DRCR, U3 SIP32431DR3-T1GE3, U4 MAX40200AUK+, U5 MAX40200AUK+, U6 RFM95_96_97_98W, U9 MICROCHIP_MCP1700T-3302E-TTMI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

Commit message: Update
Parts:
- C9: value 220uF -> 330uF
- R4: value 330R -> 180R
Changed lines of the file:
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@@
 <attribute name="NAME" x="30.5816" y="19.7358" size="0.8128" layer="25" font="vector" ratio="19" rot="R270"/>
 </element>
-<element name="R4" library="OPL_Resistor" library_urn="urn:adsk.eagle:library:8004883" package="R0402" package3d_urn="urn:adsk.eagle:package:8004940/1" value="330R" x="33.655" y="14.605" smashed="yes" rot="R180">
+<element name="R4" library="OPL_Resistor" library_urn="urn:adsk.eagle:library:8004883" package="R0402" package3d_urn="urn:adsk.eagle:package:8004940/1" value="180R" x="33.655" y="14.605" smashed="yes" rot="R180">
 <attribute name="MPN" value="RC0402JR-070RL" x="33.655" y="14.605" size="1.778" layer="27" rot="R180" display="off"/>
 <attribute name="NAME" x="33.147" y="14.986" size="0.8128" layer="25" font="vector" ratio="19" rot="R180"/>
@@
 <attribute name="VOLTAGE_RATING" value="" x="19.1008" y="12.9032" size="1.778" layer="28" rot="MR90" display="off"/>
 </element>
-<element name="C9" library="KEW_HF_V16" package="RCL_SMC_C" value="220uF" x="15.24" y="4.445" smashed="yes" rot="R270">
+<element name="C9" library="KEW_HF_V16" package="RCL_SMC_C" value="330uF" x="15.24" y="4.445" smashed="yes" rot="R270">
 <attribute name="NAME" x="15.4686" y="3.9878" size="0.8128" layer="25" font="vector" ratio="19"/>
 </element>
