File: Hardware/BT-5/BT-5.sch (EAGLE design)
At the start: 82 parts, among them J1 CORTEX_DEBUG_PTH, J2 AVR_SPI_PROG_3X22X3_LOCK, J5 JST_ZH_2PIN, U1 ATMEGA1284P-AU, U2 TPS61200DRCR, U3 SIP32431DR3-T1GE3, U4 MAX40200AUK+, U5 MAX40200AUK+, U6 RFM95_96_97_98W, U9 MICROCHIP_MCP1700T-3302E-TTMI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

Commit message: Update
Parts:
- C9: value 220uF -> 330uF
- R4: value 330R -> 180R
Other:
- note added: "330uF gives 1.5 seconds at 1.8v with MAX-7C"
Changed lines of the file:
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@@
 <part name="R3" library="OPL_Resistor" library_urn="urn:adsk.eagle:library:8004883" deviceset="SMD-RES-20K-5%-1/16W(0402)" device="" package3d_urn="urn:adsk.eagle:package:8004940/1" value="33KR"/>
 <part name="GND3" library="SparkFun-PowerSymbols" library_urn="urn:adsk.eagle:library:530" deviceset="GND" device=""/>
-<part name="R4" library="OPL_Resistor" library_urn="urn:adsk.eagle:library:8004883" deviceset="SMD-RES-20K-5%-1/16W(0402)" device="" package3d_urn="urn:adsk.eagle:package:8004940/1" value="330R"/>
+<part name="R4" library="OPL_Resistor" library_urn="urn:adsk.eagle:library:8004883" deviceset="SMD-RES-20K-5%-1/16W(0402)" device="" package3d_urn="urn:adsk.eagle:package:8004940/1" value="180R"/>
 <part name="D1" library="SparkFun-LED" library_urn="urn:adsk.eagle:library:529" deviceset="LED" device="0603" package3d_urn="urn:adsk.eagle:package:39354/1"/>
 <part name="U$2" library="GPS Antenna RainSun GPS1003-1575" deviceset="ANTENNA" device=""/>
@@
 <part name="R5" library="OPL_Resistor" library_urn="urn:adsk.eagle:library:8004883" deviceset="SMD-RES-20K-5%-1/16W(0402)" device="" package3d_urn="urn:adsk.eagle:package:8004940/1" value="330R"/>
 <part name="C11" library="Capacitor" library_urn="urn:adsk.eagle:library:16290819" deviceset="C-POL" device="ECAP-10.5MM" package3d_urn="urn:adsk.eagle:package:16290882/1" technology="_"/>
-<part name="C9" library="KEW_HF_V16" deviceset="RCL_CPOL-EU" device="SMCC" value="220uF"/>
+<part name="C9" library="KEW_HF_V16" deviceset="RCL_CPOL-EU" device="SMCC" value="330uF"/>
 <part name="D2" library="diode" library_urn="urn:adsk.eagle:library:210" deviceset="DIODE-" device="SOD123" package3d_urn="urn:adsk.eagle:package:43420/1" value="B5819W">
 <attribute name="LCSC_PART" value="C8598"/>
@@
 +20dBm 2.4v to 3.7v</text>
 <text x="335.28" y="50.8" size="1.016" layer="91" distance="60" align="top-center">4.23v / Lipo in, 3.3v out</text>
+<text x="109.22" y="144.78" size="1.016" layer="91" align="top-center">330uF gives 1.5
+seconds at 1.8v
+with MAX-7C
+</text>
 </plain>
 <instances>
@@
 <instance part="C9" gate="G$1" x="114.3" y="147.32" smashed="yes" rot="R270">
 <attribute name="NAME" x="114.7826" y="146.177" size="1.778" layer="95" rot="R270"/>
-<attribute name="VALUE" x="109.7026" y="146.177" size="1.778" layer="96" rot="R270"/>
+<attribute name="VALUE" x="117.3226" y="146.177" size="1.778" layer="96" rot="R270"/>
 </instance>
 <instance part="D2" gate="G$1" x="124.46" y="154.94" smashed="yes" rot="R180">

Commit message: Added RTTY Interrupt based code
Other:
- note added: "PS Low to enable Power Save, High to disable 4.23v out, max 18.3Mhz, Rtop 560k and Rbot 75k 3.63v out, max 15Mhz, Rtop 470k and Rbot 75k 3.37v out, max 13.3Mhz, Rtop 430k and Rbot 75k 1.83v out, max 4Mhz, Rtop 200K and Rbot 75k 0.3v to 5.5v Input"
- note removed: "PS Low to enable Power Save, High to disable 4.23v out, max 18.3Mhz, Rtop 560k and Rbot 75k 3.37v out, max 13.3Mhz, Rtop 430k and Rbot 75K 1.83v out, max 4Mhz, Rtop 200K and Rbot 75K 0.3v to 5.5v Input"
Changed lines of the file:
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@@
 <setting verticaltext="up"/>
 </settings>
-<grid distance="0.1" unitdist="inch" unit="inch" style="lines" multiple="1" display="yes" altdistance="0.05" altunitdist="inch" altunit="inch"/>
+<grid distance="0.1" unitdist="inch" unit="inch" style="lines" multiple="1" display="no" altdistance="0.01" altunitdist="inch" altunit="inch"/>
 <layers>
 <layer number="1" name="Top" color="4" fill="1" visible="no" active="no"/>
@@
 <text x="223.52" y="45.72" size="1.016" layer="91" distance="60" align="top-center">PS Low to enable Power Save, High to disable
 4.23v out, max 18.3Mhz, Rtop 560k and Rbot 75k
-3.37v out, max 13.3Mhz, Rtop 430k and Rbot 75K
-1.83v out, max 4Mhz, Rtop 200K and Rbot 75K
+3.63v out, max 15Mhz, Rtop 470k and Rbot 75k
+3.37v out, max 13.3Mhz, Rtop 430k and Rbot 75k
+1.83v out, max 4Mhz, Rtop 200K and Rbot 75k
 0.3v to 5.5v Input</text>
 <text x="86.36" y="41.91" size="1.016" layer="91" align="center">Solar Panel Mount</text>

Commit message: Updates
Other:
- note added: "Move C21 to VSS to buffer both VSolar and VBatt, remove C11 and make C21 C11 size?"
- note added: "PS Low to enable Power Save, High to disable 4.23v out, max 18.3Mhz, Rtop 560k and Rbot 75k 3.63v out, max 15Mhz, Rtop 470k and Rbot 75k 3.37v out, max 13.3Mhz, Rtop 430k and Rbot 75k 2.7v out, max 10Mhz, Rtop 330k and Rbot 75k 1.83v out, max 4Mhz, Rtop 200K and Rbot 75k 0.3v to 5.5v Input"
- note removed: "PS Low to enable Power Save, High to disable 4.23v out, max 18.3Mhz, Rtop 560k and Rbot 75k 3.63v out, max 15Mhz, Rtop 470k and Rbot 75k 3.37v out, max 13.3Mhz, Rtop 430k and Rbot 75k 1.83v out, max 4Mhz, Rtop 200K and Rbot 75k 0.3v to 5.5v Input"
Changed lines of the file:
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@@
 3.63v out, max 15Mhz, Rtop 470k and Rbot 75k
 3.37v out, max 13.3Mhz, Rtop 430k and Rbot 75k
+2.7v out, max 10Mhz, Rtop 330k and Rbot 75k
 1.83v out, max 4Mhz, Rtop 200K and Rbot 75k
 0.3v to 5.5v Input</text>
@@
 with MAX-7C
 </text>
+<text x="104.14" y="35.56" size="1.016" layer="91" distance="60" align="top-center">Move C21 to VSS to buffer both VSolar and VBatt, remove C11 and make C21 C11 size?</text>
 </plain>
 <instances>

Commit message: Updates
Parts:
- C17, C20: value 10uf -> 100KR
Changed lines of the file:
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@@
 </part>
 <part name="L1" library="OPL_Inductor" library_urn="urn:adsk.eagle:library:8004654" deviceset="SMD-INDUCTOR-3.3NH-0.3NH-300MA(0402)" device="" package3d_urn="urn:adsk.eagle:package:8004741/1" value="BLM15HD102SN1D"/>
-<part name="C17" library="OPL_Capacitor" library_urn="urn:adsk.eagle:library:8004261" deviceset="CERAMIC-10UF-6.3V-20%-X5R(0402)" device="" package3d_urn="urn:adsk.eagle:package:8004285/1" value="10uf"/>
+<part name="C17" library="OPL_Capacitor" library_urn="urn:adsk.eagle:library:8004261" deviceset="CERAMIC-10UF-6.3V-20%-X5R(0402)" device="" package3d_urn="urn:adsk.eagle:package:8004285/1" value="100KR"/>
 <part name="R11" library="OPL_Resistor" library_urn="urn:adsk.eagle:library:8004883" deviceset="SMD-RES-20K-5%-1/16W(0402)" device="" package3d_urn="urn:adsk.eagle:package:8004940/1" value="15KR"/>
 <part name="R12" library="OPL_Resistor" library_urn="urn:adsk.eagle:library:8004883" deviceset="SMD-RES-20K-5%-1/16W(0402)" device="" package3d_urn="urn:adsk.eagle:package:8004940/1" value="15KR"/>
@@
 <part name="U6" library="SparkFun-RF" library_urn="urn:adsk.eagle:library:531" deviceset="RFM69H" device="CW-433" package3d_urn="urn:adsk.eagle:package:39566/1" value="RFM95_96_97_98W"/>
 <part name="J$1" library="ESP32-Cam-Pico-V4" deviceset="SMA_EDGE" device=""/>
-<part name="C20" library="OPL_Capacitor" library_urn="urn:adsk.eagle:library:8004261" deviceset="CERAMIC-10UF-6.3V-20%-X5R(0402)" device="" package3d_urn="urn:adsk.eagle:package:8004285/1" value="10uf"/>
+<part name="C20" library="OPL_Capacitor" library_urn="urn:adsk.eagle:library:8004261" deviceset="CERAMIC-10UF-6.3V-20%-X5R(0402)" device="" package3d_urn="urn:adsk.eagle:package:8004285/1" value="100KR"/>
 <part name="B3" library="OPL_Resistor" library_urn="urn:adsk.eagle:library:8004883" deviceset="SMD-RES-20K-5%-1/16W(0402)" device="" package3d_urn="urn:adsk.eagle:package:8004940/1" value="Optional 0R Bypass"/>
 <part name="J" library="OPL_Resistor" library_urn="urn:adsk.eagle:library:8004883" deviceset="SMD-RES-20K-5%-1/16W(0402)" device="" package3d_urn="urn:adsk.eagle:package:8004940/1" value="0R"/>
